Commit message: Updated the model to have parts that can move

File: ros_ws/mowbot/models/urdf_files/mowbot_v1.urdf (robot description, URDF)
Before this commit: robot mowbot, 7 links, 6 joints
Links:
- removed link Front_left_wheel
- removed link Front_right_pivot
- removed link Front_right_wheel
- removed link Left_back_link
- removed link Right_back_link
- removed link base_link
- removed link front_left_pivot
- added link Big_Left_drive_wheel, mass 0.865783559302399; collision mesh filename=package://mowbot_v1/meshes/Big_Left_drive_wheel.STL; visual mesh filename=package://mowbot_v1/meshes/Big_Left_drive_wheel.STL
- added link Big_right_drive_wheel, mass 0.865783559302402; collision mesh filename=package://mowbot_v1/meshes/Big_right_drive_wheel.STL; visual mesh filename=package://mowbot_v1/meshes/Big_right_drive_wheel.STL
- added link Camera, mass 0.0169771128221458; collision mesh filename=package://mowbot_v1/meshes/Camera.STL; visual mesh filename=package://mowbot_v1/meshes/Camera.STL
- added link Front_left_pivot_collision, mass 0.65315365371728; collision mesh filename=package://mowbot_v1/meshes/Front_left_pivot_collision.STL; visual mesh filename=package://mowbot_v1/meshes/Front_left_pivot_collision.STL
- added link Front_left_wheel_collision, mass 0.572204494653308; collision mesh filename=package://mowbot_v1/meshes/Front_left_wheel_collision.STL; visual mesh filename=package://mowbot_v1/meshes/Front_left_wheel_collision.STL
- added link Front_right_pivot_collision, mass 0.653153653717284; collision mesh filename=package://mowbot_v1/meshes/Front_right_pivot_collision.STL; visual mesh filename=package://mowbot_v1/meshes/Front_right_pivot_collision.STL
- added link Front_right_wheel_collision, mass 0.572204494653308; collision mesh filename=package://mowbot_v1/meshes/Front_right_wheel_collision.STL; visual mesh filename=package://mowbot_v1/meshes/Front_right_wheel_collision.STL
- added link Left_back_link_collision, mass 0.457406434462016; collision mesh filename=package://mowbot_v1/meshes/Left_back_link_collision.STL; visual mesh filename=package://mowbot_v1/meshes/Left_back_link_collision.STL
- added link LiDAR, mass 0.148759159944866; collision mesh filename=package://mowbot_v1/meshes/LiDAR.STL; visual mesh filename=package://mowbot_v1/meshes/LiDAR.STL
- added link Right_back_link_collision, mass 0.457406434462017; collision mesh filename=package://mowbot_v1/meshes/Right_back_link_collision.STL; visual mesh filename=package://mowbot_v1/meshes/Right_back_link_collision.STL
- added link back_plate, mass 1.01763667439999; collision mesh filename=package://mowbot_v1/meshes/back_plate.STL; visual mesh filename=package://mowbot_v1/meshes/back_plate.STL
- added link base_link_collision, mass 8.43639227238404; collision mesh filename=package://mowbot_v1/meshes/base_link_collision.STL; visual mesh filename=package://mowbot_v1/meshes/base_link_collision.STL
- added link mow_bot_shell, mass 2.52229769150772; collision mesh filename=package://mowbot_v1/meshes/mow_bot_shell.STL; visual mesh filename=package://mowbot_v1/meshes/mow_bot_shell.STL
Joints:
- removed joint Front_left_caster_wheel
- removed joint Front_right_joint
- removed joint Left_drive_wheel
- removed joint Left_pivot_joint
- removed joint Right_caster_wheel_pivot
- added joint Front_left_caster_wheel_collision: type continuous, parent Front_left_pivot_collision, child Front_left_wheel_collision, origin xyz=-0.03569 0.0089225 -0.2032 rpy=0 0 0, axis -0.99982 -0.018718 0
- added joint Front_right_wheel_collision_joint: type continuous, parent Front_right_pivot_collision, child Front_right_wheel_collision, origin xyz=0.03569 -0.0089225 -0.2032 rpy=0 0 0, axis -0.95105 0.30902 0
- added joint Left_big_wheel: type continuous, parent Left_back_link_collision, child Big_Left_drive_wheel, origin xyz=0 -0.059347 0 rpy=0 0 -3.1416, axis 0 1 0
- added joint Left_drive_wheel_collision: type revolute, parent base_link_collision, child Left_back_link_collision, origin xyz=-1.5558 -0.024 0.62929 rpy=0 0 3.1416, axis 0 1 0, limit effort=14.08 velocity=12.47
- added joint LiDAR_unit: type revolute, parent mow_bot_shell, child LiDAR, origin xyz=0.13767 0 0.064668 rpy=0 0 0, axis 0 0 0, limit lower=0 upper=0 effort=0 velocity=0
- added joint Right_caster_wheel_pivot_collision: type continuous, parent base_link_collision, child Front_right_pivot_collision, origin xyz=-0.45126 -0.88591 0.73883 rpy=0 0 0, axis 0 0 -1
- added joint Right_drive_wheel_collision: type revolute, parent base_link_collision, child Right_back_link_collision, origin xyz=-1.5558 -0.9108 0.62929 rpy=0 0 -1.5708, axis -1 0 0, limit effort=14.08 velocity=12.47
- added joint camera_box: type revolute, parent mow_bot_shell, child Camera, origin xyz=0.21869 0 0 rpy=0 0 3.1416, axis 0 0 0, limit lower=0 upper=0 effort=0 velocity=0
- added joint left_caster_wheel_pivot_collision: type continuous, parent base_link_collision, child Front_left_pivot_collision, origin xyz=-0.45126 -0.04771 0.73883 rpy=0 0 -1.5708, axis 0 0 -1
- added joint mowbot_back: type fixed, parent base_link_collision, child back_plate, origin xyz=-1.6501 -0.46681 0.64993 rpy=0 0 0, axis 0 0 0
- added joint shell_main: type fixed, parent base_link_collision, child mow_bot_shell, origin xyz=-1.4447 -0.46681 0.81909 rpy=0 0 0, axis 0 0 0
- joint Right_drive_wheel: axis -1 0 0 -> 0 -1 0; child Right_back_link -> Big_right_drive_wheel; limit effort=14.08 velocity=12.47 -> (none); origin xyz=-1.5557647261818 -0.910799826679582 0.637929355601164 rpy=0 0 -1.5707963267949 -> xyz=0.059347 0 0 rpy=0 0 1.5708; parent base_link -> Right_back_link_collision; type fixed -> continuous
